File: qfbms32 ai pcb/qfbms32.kicad_pcb (KiCad board)
At the start: 2 copper layers, 130 x 32 mm, 107 parts, among them Q1 AGM15T03LL, Q2 AGM15T03LL, U4 LTC7138, U7 ISO1050 (DUB-8)

Commit message: feat: add qfbms32 AI PCB design files, scratch scripts, and dashboard tools
Parts:
- removed C_S1, C_S2: 100nF, C_0603_1608Metric
- added C_SSR1: 100nF, C_0603_1608Metric, F.Cu at (28.4, 1.75)
- added C_SSR2: 1uF, C_0805_2012Metric, F.Cu at (30.0, 1.70)
- added FB1: Unmarked, R_0603_1608Metric, F.Cu at (30.9, 26.6)
- added R_CHG2: 2203, R_0805_2012Metric, F.Cu at (15.2, 1.10)
- added R_DSG1: 1000, R_0805_2012Metric, F.Cu at (30.8, 29.8)
- added R_G1: 01X, R_0603_1608Metric, F.Cu at (29.5, 7.60)
- added R_GS1: 474, R_0603_1608Metric, F.Cu at (29.5, 8.95)
- added R_S1: 1000, R_0805_2012Metric, F.Cu at (17.6, 15.0)
- added R_S2: 1000, R_0805_2012Metric, F.Cu at (17.5, 17.0)
- added R_SEC1: 01X, R_0603_1608Metric, F.Cu at (29.8, 17.2)
- added R_SSR1: 01X, R_0603_1608Metric, F.Cu at (29.2, 4.05)
- F1: value JT 18A -> JT 15A
- moved F1 2.10 mm to (17.4, 27.5)
