File: qfbms32 ai pcb/qfbms32.kicad_pcb (KiCad board)
At the start: 2 copper layers, 130 x 32 mm, 116 parts, among them Q1 AGM15T03LL, Q2 AGM15T03LL, U4 LTC7138, U7 ISO1050 (DUB-8)

Commit message: Snapshot qfbms32 placement-clone work before forking lookalike vs working paths.
Includes board/sch updates, new reference photos, dashboard tweaks, and scratch placement scripts; leaves the new qfbms32 fork/ tree uncommitted.

Co-authored-by: Cursor <cursoragent@cursor.com>
Parts:
- added D_GS1: PDZ16B, D_SOD-323, F.Cu at (29.2, 10.8)
- added R_SSR2: 10k, R_0603_1608Metric, F.Cu at (29.1, 5.70)
