File: qfbms32 ai pcb/qfbms32.kicad_pcb (KiCad board)
At the start: 2 copper layers, 130 x 32 mm, 118 parts, among them Q1 AGM15T03LL, Q2 AGM15T03LL, U4 LTC7138, U7 ISO1050 (DUB-8)

Commit message: update qfbms32 ai pcb info
Parts:
- added C_F1: 0.22uF, C_0402_1005Metric, F.Cu at (82.2, 18.5)
- added C_F10: 0.22uF, C_0402_1005Metric, F.Cu at (78.9, 11.9)
- added C_F11: 0.22uF, C_0402_1005Metric, F.Cu at (79.9, 11.9)
- added C_F12: 0.22uF, C_0402_1005Metric, F.Cu at (81.6, 13.5)
- added C_F13: 0.22uF, C_0402_1005Metric, F.Cu at (81.5, 12.4)
- added C_F14: 0.22uF, C_0402_1005Metric, F.Cu at (81.5, 11.2)
- added C_F15: 0.22uF, C_0402_1005Metric, F.Cu at (81.7, 10.1)
- added C_F16: 0.22uF, C_0402_1005Metric, F.Cu at (82.7, 8.12)
- added C_F17: 0.22uF, C_0402_1005Metric, F.Cu at (39.1, 18.5)
- added C_F18: 0.22uF, C_0402_1005Metric, F.Cu at (37.9, 18.4)
- added C_F19: 0.22uF, C_0402_1005Metric, F.Cu at (39.0, 16.5)
- added C_F2: 0.22uF, C_0402_1005Metric, F.Cu at (81.0, 18.4)
- added C_F20: 0.22uF, C_0402_1005Metric, F.Cu at (38.0, 16.4)
- added C_F21: 0.22uF, C_0402_1005Metric, F.Cu at (37.0, 16.4)
- added C_F22: 0.22uF, C_0402_1005Metric, F.Cu at (38.4, 14.9)
- added C_F23: 0.22uF, C_0402_1005Metric, F.Cu at (37.0, 14.4)
- added C_F24: 0.22uF, C_0402_1005Metric, F.Cu at (38.5, 13.8)
- added C_F25: 0.22uF, C_0402_1005Metric, F.Cu at (35.8, 14.1)
- added C_F26: 0.22uF, C_0402_1005Metric, F.Cu at (34.8, 13.9)
- added C_F27: 0.22uF, C_0402_1005Metric, F.Cu at (35.8, 12.1)
- added C_F28: 0.22uF, C_0402_1005Metric, F.Cu at (36.9, 12.3)
- added C_F29: 0.22uF, C_0402_1005Metric, F.Cu at (38.4, 12.6)
- added C_F3: 0.22uF, C_0402_1005Metric, F.Cu at (82.1, 16.5)
- added C_F30: 0.22uF, C_0402_1005Metric, F.Cu at (38.4, 11.4)
- added C_F31: 0.22uF, C_0402_1005Metric, F.Cu at (38.6, 10.3)
- added C_F32: 0.22uF, C_0402_1005Metric, F.Cu at (39.0, 8.72)
- added C_F4: 0.22uF, C_0402_1005Metric, F.Cu at (79.9, 18.4)
- added C_F5: 0.22uF, C_0402_1005Metric, F.Cu at (80.7, 16.8)
- added C_F6: 0.22uF, C_0402_1005Metric, F.Cu at (80.5, 15.7)
- added C_F7: 0.22uF, C_0402_1005Metric, F.Cu at (81.5, 14.6)
- added C_F8: 0.22uF, C_0402_1005Metric, F.Cu at (80.0, 14.2)
- added C_F9: 0.22uF, C_0402_1005Metric, F.Cu at (78.9, 13.9)
- R_F1, R_F10, R_F11, R_F12, R_F13, R_F14, R_F15, R_F16, R_F17, R_F18, R_F19, R_F2, R_F20, R_F21, R_F22, R_F23, R_F24, R_F25, R_F26, R_F27, R_F28, R_F29, R_F3, R_F30, R_F31, R_F32, R_F4, R_F5, R_F6, R_F7, R_F8, R_F9: value 100R -> 20R
Connections:
- C_SSR1 pad 1: (no net) -> VBOOST
- C_SSR1 pad 2: (no net) -> GND
- C_SSR2 pad 1: (no net) -> VBOOST
- C_SSR2 pad 2: (no net) -> GND
- D_GS1 pad 1: (no net) -> Q1_GATE
- D_GS1 pad 2: (no net) -> CHG+
- F1 pad 1: (no net) -> CELL32
- F1 pad 2: (no net) -> CELL32_FUSED
- J_BAT1 pad 1: (no net) -> CELL32
- J_BAT1 pad 2: (no net) -> CELL0
- J_CELL1 pad 1: (no net) -> CELL9
- J_CELL1 pad 10: (no net) -> CELL0
- J_CELL1 pad 2: (no net) -> CELL8
- J_CELL1 pad 3: (no net) -> CELL7
- J_CELL1 pad 4: (no net) -> CELL6
- J_CELL1 pad 5: (no net) -> CELL5
- J_CELL1 pad 6: (no net) -> CELL4
- J_CELL1 pad 7: (no net) -> CELL3
- J_CELL1 pad 8: (no net) -> CELL2
- J_CELL1 pad 9: (no net) -> CELL1
- J_CELL2 pad 1: (no net) -> CELL18
- J_CELL2 pad 2: (no net) -> CELL17
- J_CELL2 pad 3: (no net) -> CELL16
- J_CELL2 pad 4: (no net) -> CELL15
- J_CELL2 pad 5: (no net) -> CELL14
- J_CELL2 pad 6: (no net) -> CELL13
- J_CELL2 pad 7: (no net) -> CELL12
- J_CELL2 pad 8: (no net) -> CELL11
- J_CELL2 pad 9: (no net) -> CELL10
- J_CELL3 pad 1: (no net) -> CELL26
- J_CELL3 pad 2: (no net) -> CELL25
- J_CELL3 pad 3: (no net) -> CELL24
- J_CELL3 pad 4: (no net) -> CELL23
- J_CELL3 pad 5: (no net) -> CELL22
- J_CELL3 pad 6: (no net) -> CELL21
- J_CELL3 pad 7: (no net) -> CELL20
- J_CELL3 pad 8: (no net) -> CELL19
- J_CELL4 pad 1: (no net) -> CELL32
- J_CELL4 pad 2: (no net) -> CELL31
- J_CELL4 pad 3: (no net) -> CELL30
- J_CELL4 pad 4: (no net) -> CELL29
- J_CELL4 pad 5: (no net) -> CELL28
- J_CELL4 pad 6: (no net) -> CELL27
- J_CHG1 pad 1: (no net) -> CHG+
- J_CHG1 pad 2: (no net) -> CHG-
- J_COMM1 pad 1: (no net) -> CANH
- J_COMM1 pad 2: (no net) -> CANL
- J_COMM1 pad 3: (no net) -> ISO_GND
- J_COMM1 pad 4: (no net) -> 5VExt
- J_T1 pad 1: (no net) -> TS1
- J_T1 pad 2: (no net) -> GND
- J_T2 pad 1: (no net) -> TS2
- J_T2 pad 2: (no net) -> GND
- J_T3 pad 1: (no net) -> TS3
- J_T3 pad 2: (no net) -> GND
- J_T4 pad 1: (no net) -> TS4
- J_T4 pad 2: (no net) -> GND
- Q1 pad 1: (no net) -> Q1_GATE
- Q1 pad 2: (no net) -> CHG+
- Q1 pad 3: (no net) -> CHG+
- Q1 pad 4: (no net) -> CHG+
- Q1 pad 5: (no net) -> CHG+
- Q1 pad 6: (no net) -> CHG+
- Q1 pad 7: (no net) -> CHG+
- Q1 pad 8: (no net) -> CHG+
- Q1 pad D: (no net) -> CELL32_FUSED
- Q2 pad 1: (no net) -> Q2_GATE
- Q2 pad 2: (no net) -> PACK+
- Q2 pad 3: (no net) -> PACK+
- Q2 pad 4: (no net) -> PACK+
- Q2 pad 5: (no net) -> PACK+
- Q2 pad 6: (no net) -> PACK+
- Q2 pad 7: (no net) -> PACK+
- Q2 pad 8: (no net) -> PACK+
- Q2 pad D: (no net) -> CELL32_FUSED
- R_F1 pad 1: (no net) -> CELL32
- R_F1 pad 2: (no net) -> BQ2_VC16
- R_F10 pad 1: (no net) -> CELL23
- R_F10 pad 2: (no net) -> BQ2_VC7
- R_F11 pad 1: (no net) -> CELL22
- R_F11 pad 2: (no net) -> BQ2_VC6
- R_F12 pad 1: (no net) -> CELL21
- R_F12 pad 2: (no net) -> BQ2_VC5
- R_F13 pad 1: (no net) -> CELL20
- R_F13 pad 2: (no net) -> BQ2_VC4
- R_F14 pad 1: (no net) -> CELL19
- R_F14 pad 2: (no net) -> BQ2_VC3
- R_F15 pad 1: (no net) -> CELL18
- R_F15 pad 2: (no net) -> BQ2_VC2
- R_F16 pad 1: (no net) -> CELL17
- R_F16 pad 2: (no net) -> BQ2_VC1
- R_F17 pad 1: (no net) -> CELL16
- R_F17 pad 2: (no net) -> BQ1_VC16
- R_F18 pad 1: (no net) -> CELL15
- R_F18 pad 2: (no net) -> BQ1_VC15
- R_F19 pad 1: (no net) -> CELL14
- R_F19 pad 2: (no net) -> BQ1_VC14
- R_F2 pad 1: (no net) -> CELL31
- R_F2 pad 2: (no net) -> BQ2_VC15
- R_F20 pad 1: (no net) -> CELL13
- R_F20 pad 2: (no net) -> BQ1_VC13
- R_F21 pad 1: (no net) -> CELL12
- R_F21 pad 2: (no net) -> BQ1_VC12
- R_F22 pad 1: (no net) -> CELL11
- R_F22 pad 2: (no net) -> BQ1_VC11
- R_F23 pad 1: (no net) -> CELL10
- R_F23 pad 2: (no net) -> BQ1_VC10
- R_F24 pad 1: (no net) -> CELL9
- R_F24 pad 2: (no net) -> BQ1_VC9
- R_F25 pad 1: (no net) -> CELL8
- R_F25 pad 2: (no net) -> BQ1_VC8
- R_F26 pad 1: (no net) -> CELL7
- R_F26 pad 2: (no net) -> BQ1_VC7
- R_F27 pad 1: (no net) -> CELL6
- R_F27 pad 2: (no net) -> BQ1_VC6
- R_F28 pad 1: (no net) -> CELL5
- R_F28 pad 2: (no net) -> BQ1_VC5
- R_F29 pad 1: (no net) -> CELL4
- R_F29 pad 2: (no net) -> BQ1_VC4
- R_F3 pad 1: (no net) -> CELL30
- R_F3 pad 2: (no net) -> BQ2_VC14
- R_F30 pad 1: (no net) -> CELL3
- R_F30 pad 2: (no net) -> BQ1_VC3
- R_F31 pad 1: (no net) -> CELL2
- R_F31 pad 2: (no net) -> BQ1_VC2
- R_F32 pad 1: (no net) -> CELL1
- R_F32 pad 2: (no net) -> BQ1_VC1
- R_F4 pad 1: (no net) -> CELL29
- R_F4 pad 2: (no net) -> BQ2_VC13
- R_F5 pad 1: (no net) -> CELL28
- R_F5 pad 2: (no net) -> BQ2_VC12
- R_F6 pad 1: (no net) -> CELL27
- R_F6 pad 2: (no net) -> BQ2_VC11
- R_F7 pad 1: (no net) -> CELL26
- R_F7 pad 2: (no net) -> BQ2_VC10
- R_F8 pad 1: (no net) -> CELL25
- R_F8 pad 2: (no net) -> BQ2_VC9
- R_F9 pad 1: (no net) -> CELL24
- R_F9 pad 2: (no net) -> BQ2_VC8
- R_G1 pad 1: (no net) -> Q1_GATE
- R_G1 pad 2: (no net) -> SSR_OUT_CHG
- R_GS1 pad 1: (no net) -> Q1_GATE
- R_GS1 pad 2: (no net) -> CHG+
- R_SH1 pad 1: (no net) -> CELL0
- R_SH1 pad 2: (no net) -> SHUNT_MID
- R_SH2 pad 1: (no net) -> SHUNT_MID
- R_SH2 pad 2: (no net) -> CHG-
- R_SSR1 pad 1: (no net) -> SSR_OUT_CHG
- R_SSR1 pad 2: (no net) -> Q1_GATE
- R_SSR2 pad 1: (no net) -> Q1_GATE
- R_SSR2 pad 2: (no net) -> GND
- U_BQ1 pad 1: (no net) -> BQ1_VC15
- U_BQ1 pad 10: (no net) -> BQ1_VC6
- U_BQ1 pad 11: (no net) -> BQ1_VC5
- U_BQ1 pad 12: (no net) -> BQ1_VC4
- U_BQ1 pad 13: (no net) -> BQ1_VC3
- U_BQ1 pad 14: (no net) -> BQ1_VC2
- U_BQ1 pad 15: (no net) -> BQ1_VC1
- U_BQ1 pad 16: (no net) -> CELL0
- U_BQ1 pad 17: (no net) -> GND
- U_BQ1 pad 18: (no net) -> SRP
- U_BQ1 pad 2: (no net) -> BQ1_VC14
- U_BQ1 pad 20: (no net) -> SRN
- U_BQ1 pad 21: (no net) -> TS1
- U_BQ1 pad 22: (no net) -> TS2
- U_BQ1 pad 23: (no net) -> TS3
- U_BQ1 pad 3: (no net) -> BQ1_VC13
- U_BQ1 pad 4: (no net) -> BQ1_VC12
- U_BQ1 pad 47: (no net) -> BQ1_BAT
- U_BQ1 pad 48: (no net) -> BQ1_VC16
- U_BQ1 pad 5: (no net) -> BQ1_VC11
- U_BQ1 pad 6: (no net) -> BQ1_VC10
- U_BQ1 pad 7: (no net) -> BQ1_VC9
- U_BQ1 pad 8: (no net) -> BQ1_VC8
- U_BQ1 pad 9: (no net) -> BQ1_VC7
- U_BQ2 pad 1: (no net) -> BQ2_VC15
- U_BQ2 pad 10: (no net) -> BQ2_VC6
- U_BQ2 pad 11: (no net) -> BQ2_VC5
- U_BQ2 pad 12: (no net) -> BQ2_VC4
- U_BQ2 pad 13: (no net) -> BQ2_VC3
- U_BQ2 pad 14: (no net) -> BQ2_VC2
- U_BQ2 pad 15: (no net) -> BQ2_VC1
- U_BQ2 pad 16: (no net) -> CELL16
- U_BQ2 pad 17: (no net) -> GND
- U_BQ2 pad 18: (no net) -> SRP
- U_BQ2 pad 2: (no net) -> BQ2_VC14
- U_BQ2 pad 20: (no net) -> SRN
- U_BQ2 pad 21: (no net) -> TS4
- U_BQ2 pad 3: (no net) -> BQ2_VC13
- U_BQ2 pad 4: (no net) -> BQ2_VC12
- U_BQ2 pad 47: (no net) -> BQ2_BAT
- U_BQ2 pad 48: (no net) -> BQ2_VC16
- U_BQ2 pad 5: (no net) -> BQ2_VC11
- U_BQ2 pad 6: (no net) -> BQ2_VC10
- U_BQ2 pad 7: (no net) -> BQ2_VC9
- U_BQ2 pad 8: (no net) -> BQ2_VC8
- U_BQ2 pad 9: (no net) -> BQ2_VC7
- U_SSR1 pad 1: (no net) -> PIN_CHG_EN
- U_SSR1 pad 2: (no net) -> PIN_OUT_EN
- U_SSR1 pad 3: (no net) -> PIN_PSW_EN
- U_SSR1 pad 4: (no net) -> GND
- U_SSR1 pad 5: (no net) -> VBOOST
- U_SSR1 pad 6: (no net) -> CELL32
Routing:
- net CELL32: track 0.00 -> 16.9 mm
- net GND: track 0.00 -> 14.7 mm
- net CELL1: track 0.00 -> 11.2 mm
- net CELL2: track 0.00 -> 10.4 mm
- net CELL26: track 0.00 -> 9.67 mm
- net CELL3: track 0.00 -> 9.65 mm
- net CELL31: track 0.00 -> 9.08 mm
- net CELL25: track 0.00 -> 8.91 mm
- net CELL10: track 0.00 -> 8.91 mm
- net CELL4: track 0.00 -> 8.90 mm
- net CELL30: track 0.00 -> 8.33 mm
- net CELL18: track 0.00 -> 8.22 mm
- net CELL24: track 0.00 -> 8.16 mm
- net CELL11: track 0.00 -> 8.15 mm
- net CELL5: track 0.00 -> 8.15 mm
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