File: qfbms32 ai pcb/qfbms32.kicad_sch (KiCad schematic)
At the start: 19 parts, among them Q1 AGM15T03LL (CHG FET), Q2 AGM15T03LL (DSG FET), U1 BQ7695202 (IC1 - Lower 16S), U2 BQ7695202 (IC2 - Upper 16S), U3 ESP32-C3-MINI-1, U7 ISO1050 (Isolated CAN Transce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

Commit message: Snapshot qfbms32 placement-clone work before forking lookalike vs working paths.
Includes board/sch updates, new reference photos, dashboard tweaks, and scratch placement scripts; leaves the new qfbms32 fork/ tree uncommitted.

Co-authored-by: Cursor <cursoragent@cursor.com>
Parts:
- added D_GS1: PDZ16B, Diode_SMD:D_SOD-323, symbol Device:D_Zener
- added R_SSR2: 10k, Resistor_SMD:R_0603_1608Metric, symbol Device:R
Changed lines of the file:
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@@
+		)
+	)
+	(symbol (lib_id "Device:D_Zener")
+		(at 185.0 25.0 0)
+		(unit 1)
+		(exclude_from_sim no)
+		(in_bom yes)
+		(on_board yes)
+		(dnp no)
+		(property "Reference" "D_GS1" (at 185.0 21.0 0) (effects (font (size 1.27 1.27))))
+		(property "Value" "PDZ16B" (at 185.0 29.0 0) (effects (font (size 1.27 1.27))))
+		(property "Footprint" "Diode_SMD:D_SOD-323" (at 185.0 25.0 0) (hide yes) (effects (font (size 1.27 1.27))))
+		(pin "1")
+		(pin "2")
+		(instances
+			(project "qfbms32"
+				(path "/a2322edc-ff52-449c-92df-24faffac0236" (reference "D_GS1") (unit 1))
+			)
+		)
+	)
+	(symbol (lib_id "Device:R")
+		(at 185.0 35.0 0)
+		(unit 1)
+		(exclude_from_sim no)
+		(in_bom yes)
+		(on_board yes)
+		(dnp no)
+		(property "Reference" "R_SSR2" (at 185.0 31.0 0) (effects (font (size 1.27 1.27))))
+		(property "Value" "10k" (at 185.0 39.0 0) (effects (font (size 1.27 1.27))))
+		(property "Footprint" "Resistor_SMD:R_0603_1608Metric" (at 185.0 35.0 0) (hide yes) (effects (font (size 1.27 1.27))))
+		(pin "1")
+		(pin "2")
+		(instances
+			(project "qfbms32"
+				(path "/a2322edc-ff52-449c-92df-24faffac0236" (reference "R_SSR2") (unit 1))
+			)
 		)
 	)
