File: qfbms32 ai pcb/qfbms32.kicad_sch (KiCad schematic)
At the start: 21 parts, among them Q1 AGM15T03LL (CHG FET), Q2 AGM15T03LL (DSG FET), U1 BQ7695202 (IC1 - Lower 16S), U2 BQ7695202 (IC2 - Upper 16S), U3 ESP32-C3-MINI-1, U7 ISO1050 (Isolated CAN Transce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

Commit message: update qfbms32 ai pcb info
Parts:
- added C_F1, C_F10, C_F11, C_F12, C_F13, C_F14, C_F15, C_F16, C_F17, C_F18, C_F19, C_F2, C_F20, C_F21, C_F22, C_F23, C_F24, C_F25, C_F26, C_F27, C_F28, C_F29, C_F3, C_F30, C_F31, C_F32, C_F4, C_F5, C_F6, C_F7, C_F8, C_F9: 0.22uF, Capacitor_SMD:C_0402_1005Metric, symbol Device:C
- added F1: 15A, Fuse:Fuse_2512_6332Metric, symbol Device:R
- added J_BAT1: XT30 BAT, qfbms:XT30PW-M_Lugs, symbol Connector_Generic:Conn_01x02
- added J_CELL1: J_CELL1, Connector_JST:JST_GH_BM10B-GHS-TBT_1x10-1MP_P1.25mm_Vertical, symbol Connector_Generic:Conn_01x10
- added J_CELL2: J_CELL2, Connector_JST:JST_GH_BM09B-GHS-TBT_1x09-1MP_P1.25mm_Vertical, symbol Connector_Generic:Conn_01x09
- added J_CELL3: J_CELL3, Connector_JST:JST_GH_BM08B-GHS-TBT_1x08-1MP_P1.25mm_Vertical, symbol Connector_Generic:Conn_01x08
- added J_CELL4: J_CELL4, Connector_JST:JST_GH_BM06B-GHS-TBT_1x06-1MP_P1.25mm_Vertical, symbol Connector_Generic:Conn_01x06
- added J_CHG1: XT30 CHG, qfbms:XT30PW-F_Lugs, symbol Connector_Generic:Conn_01x02
- added J_COMM1: CAN/5V, Connector_JST:JST_GH_BM04B-GHS-TBT_1x04-1MP_P1.25mm_Vertical, symbol Connector_Generic:Conn_01x04
- added J_T1: T1, Connector_JST:JST_GH_BM02B-GHS-TBT_1x02-1MP_P1.25mm_Vertical, symbol Connector_Generic:Conn_01x02
- added J_T2: T2, Connector_JST:JST_GH_BM02B-GHS-TBT_1x02-1MP_P1.25mm_Vertical, symbol Connector_Generic:Conn_01x02
- added J_T3: T3, Connector_JST:JST_GH_BM02B-GHS-TBT_1x02-1MP_P1.25mm_Vertical, symbol Connector_Generic:Conn_01x02
- added J_T4: T4, Connector_JST:JST_GH_BM02B-GHS-TBT_1x02-1MP_P1.25mm_Vertical, symbol Connector_Generic:Conn_01x02
- added R_F1, R_F10, R_F11, R_F12, R_F13, R_F14, R_F15, R_F16, R_F17, R_F18, R_F19, R_F2, R_F20, R_F21, R_F22, R_F23, R_F24, R_F25, R_F26, R_F27, R_F28, R_F29, R_F3, R_F30, R_F31, R_F32, R_F4, R_F5, R_F6, R_F7, R_F8, R_F9: 20R, Resistor_SMD:R_0402_1005Metric, symbol Device:R
- added R_SH1, R_SH2: R001, Resistor_SMD:R_2512_6332Metric, symbol Device:R
- added R_SSR1: 01X, Resistor_SMD:R_0603_1608Metric, symbol Device:R
- renumbered U1 to U_BQ1, U2 to U_BQ2, U3 to U_ESP1
Connections:
- net 5VExt: now also J_COMM1.4 (Pin_4)
- net CANH: now also J_COMM1.1 (Pin_1)
- net CANL: now also J_COMM1.2 (Pin_2)
- net GND: now also C_SSR1.2, C_SSR2.2, R_SSR2.2, U_BQ1.17 (VSS), U_BQ1.33 (RST_SHUT), U_BQ2.17 (VSS), U_BQ2.33 (RST_SHUT), U_SSR1.4 (GND), J_T1.2 (Pin_2), J_T2.2 (Pin_2), J_T3.2 (Pin_2), J_T4.2 (Pin_2)
- net I2C_SDA: now also U_BQ1.27 (SDA/SPI_MISO), U_BQ2.27 (SDA/SPI_MISO)
- net ISO_GND: now also J_COMM1.3 (Pin_3)
- net PIN_CHG_EN: now also U_SSR1.1 (IN_CHG)
- net PIN_OUT_EN: now also U_SSR1.2 (IN_DSG)
- net PIN_PSW_EN: now also U_SSR1.3 (PSW_EN)
- net VBOOST: now reaches C_SSR1.1
- net VBOOST: now also C_SSR2.1, U_SSR1.5 (VBOOST)
- net Q1_GATE: now reaches R_SSR2.1
- net Q1_GATE: now also Q1.1 (G), R_G1.2, R_SSR1.2
- net CELL32: now reaches U_SSR1.6 (VBAT_S)
- net CELL32: now also F1.1, J_BAT1.1 (Pin_1), J_CELL4.1 (Pin_1), R_F1.2
- net SSR_OUT_DSG: now reaches U_SSR1.7 (OUT_DSG)
- net SSR_OUT_DSG: now also R_G2.1
- net SSR_OUT_CHG: now reaches U_SSR1.8 (OUT_CHG)
- net SSR_OUT_CHG: now also R_G1.1, R_SSR1.1
- net Q2_GATE: now reaches R_G2.2
- net Q2_GATE: now also Q2.1 (G)
- net PACK+: now reaches Q2.2 (S)
- net CELL32_FUSED: now reaches Q2.D
- net CELL32_FUSED: now also Q1.D, F1.2
- net BQ2_VC15: now reaches U_BQ2.1 (VC15)
- net BQ2_VC15: now also C_F31.2, C_F32.1, R_F2.1
- net BQ2_VC6: now reaches U_BQ2.10 (VC6)
- net BQ2_VC6: now also C_F22.2, C_F23.1, R_F11.1
- net BQ2_VC5: now reaches U_BQ2.11 (VC5)
- net BQ2_VC5: now also C_F21.2, C_F22.1, R_F12.1
- net BQ2_VC4: now reaches U_BQ2.12 (VC4)
- net BQ2_VC4: now also C_F20.2, C_F21.1, R_F13.1
- net BQ2_VC3: now reaches U_BQ2.13 (VC3)
- net BQ2_VC3: now also C_F19.2, C_F20.1, R_F14.1
- net BQ2_VC2: now reaches U_BQ2.14 (VC2)
- net BQ2_VC2: now also C_F18.2, C_F19.1, R_F15.1
- net BQ2_VC1: now reaches U_BQ2.15 (VC1)
- net BQ2_VC1: now also C_F17.2, C_F18.1, R_F16.1
- net CELL16: now reaches U_BQ2.16 (VC0)
- net CELL16: now also C_F17.1, J_CELL2.3 (Pin_3), R_F17.2
- net SRP: now reaches U_BQ2.18 (SRP)
- net SRP: now also U_BQ1.18 (SRP)
- net BQ2_VC14: now reaches U_BQ2.2 (VC14)
- net BQ2_VC14: now also C_F30.2, C_F31.1, R_F3.1
- net SRN: now reaches U_BQ2.20 (SRN)
- net SRN: now also U_BQ1.20 (SRN)
- net TS4: now reaches U_BQ2.21 (TS1)
- net TS4: now also J_T4.1 (Pin_1)
- net I2C_SCL: now reaches U_BQ2.26 (SCL/SPI_CLK)
- net I2C_SCL: now also U_BQ1.26 (SCL/SPI_CLK)
- net BQ2_VC13: now reaches U_BQ2.3 (VC13)
- net BQ2_VC13: now also C_F29.2, C_F30.1, R_F4.1
- net BQ2_VC12: now reaches U_BQ2.4 (VC12)
- net BQ2_VC12: now also C_F28.2, C_F29.1, R_F5.1
- net BQ2_VC16: now reaches U_BQ2.47 (BAT)
- net BQ2_VC16: now also U_BQ2.48 (VC16), C_F32.2, R_F1.1
- net BQ2_VC11: now reaches U_BQ2.5 (VC11)
- net BQ2_VC11: now also C_F27.2, C_F28.1, R_F6.1
- net BQ2_VC10: now reaches U_BQ2.6 (VC10)
- net BQ2_VC10: now also C_F26.2, C_F27.1, R_F7.1
- net BQ2_VC9: now reaches U_BQ2.7 (VC9)
- net BQ2_VC9: now also C_F25.2, C_F26.1, R_F8.1
- net BQ2_VC8: now reaches U_BQ2.8 (VC8)
- net BQ2_VC8: now also C_F24.2, C_F25.1, R_F9.1
- net BQ2_VC7: now reaches U_BQ2.9 (VC7)
- net BQ2_VC7: now also C_F23.2, C_F24.1, R_F10.1
- net CHG+: now reaches Q1.2 (S)
- net CHG+: now also J_CHG1.1 (Pin_1)
- net BQ1_VC15: now reaches U_BQ1.1 (VC15)
- net BQ1_VC15: now also C_F15.2, C_F16.1, R_F18.1
- net BQ1_VC6: now reaches U_BQ1.10 (VC6)
- net BQ1_VC6: now also C_F6.2, C_F7.1, R_F27.1
- net BQ1_VC5: now reaches U_BQ1.11 (VC5)
- net BQ1_VC5: now also C_F5.2, C_F6.1, R_F28.1
- net BQ1_VC4: now reaches U_BQ1.12 (VC4)
- net BQ1_VC4: now also C_F4.2, C_F5.1, R_F29.1
- net BQ1_VC3: now reaches U_BQ1.13 (VC3)
- net BQ1_VC3: now also C_F3.2, C_F4.1, R_F30.1
- net BQ1_VC2: now reaches U_BQ1.14 (VC2)
- net BQ1_VC2: now also C_F2.2, C_F3.1, R_F31.1
- net BQ1_VC1: now reaches U_BQ1.15 (VC1)
- net BQ1_VC1: now also C_F1.2, C_F2.1, R_F32.1
- net CELL0: now reaches U_BQ1.16 (VC0)
- net CELL0: now also C_F1.1, J_BAT1.2 (Pin_2), J_CELL1.10 (Pin_10), R_SH1.1
- net BQ1_VC14: now reaches U_BQ1.2 (VC14)
- net BQ1_VC14: now also C_F14.2, C_F15.1, R_F19.1
- net TS1: now reaches U_BQ1.21 (TS1)
- net TS1: now also J_T1.1 (Pin_1)
- net TS2: now reaches U_BQ1.22 (TS2/WAKE)
- net TS2: now also J_T2.1 (Pin_1)
- net TS3: now reaches U_BQ1.23 (TS3)
- net TS3: now also J_T3.1 (Pin_1)
- net BQ1_VC13: now reaches U_BQ1.3 (VC13)
- net BQ1_VC13: now also C_F13.2, C_F14.1, R_F20.1
- net BQ1_VC12: now reaches U_BQ1.4 (VC12)
- net BQ1_VC12: now also C_F12.2, C_F13.1, R_F21.1
- net BQ1_VC16: now reaches U_BQ1.47 (BAT)
- net BQ1_VC16: now also U_BQ1.48 (VC16), C_F16.2, R_F17.1
- net BQ1_VC11: now reaches U_BQ1.5 (VC11)
- net BQ1_VC11: now also C_F11.2, C_F12.1, R_F22.1
- net BQ1_VC10: now reaches U_BQ1.6 (VC10)
- net BQ1_VC10: now also C_F10.2, C_F11.1, R_F23.1
- net BQ1_VC9: now reaches U_BQ1.7 (VC9)
- net BQ1_VC9: now also C_F10.1, C_F9.2, R_F24.1
- net BQ1_VC8: now reaches U_BQ1.8 (VC8)
- net BQ1_VC8: now also C_F8.2, C_F9.1, R_F25.1
- net BQ1_VC7: now reaches U_BQ1.9 (VC7)
- net BQ1_VC7: now also C_F7.2, C_F8.1, R_F26.1
- new net CELL1: J_CELL1.9 (Pin_9), R_F32.2
- new net CELL10: J_CELL2.9 (Pin_9), R_F23.2
- new net CELL11: J_CELL2.8 (Pin_8), R_F22.2
- new net CELL12: J_CELL2.7 (Pin_7), R_F21.2
- new net CELL13: J_CELL2.6 (Pin_6), R_F20.2
- new net CELL14: J_CELL2.5 (Pin_5), R_F19.2
- new net CELL15: J_CELL2.4 (Pin_4), R_F18.2
- new net CELL17: J_CELL2.2 (Pin_2), R_F16.2
- new net CELL18: J_CELL2.1 (Pin_1), R_F15.2
- new net CELL19: J_CELL3.8 (Pin_8), R_F14.2
- new net CELL2: J_CELL1.8 (Pin_8), R_F31.2
- new net CELL20: J_CELL3.7 (Pin_7), R_F13.2
- new net CELL21: J_CELL3.6 (Pin_6), R_F12.2
- new net CELL22: J_CELL3.5 (Pin_5), R_F11.2
- new net CELL23: J_CELL3.4 (Pin_4), R_F10.2
- new net CELL24: J_CELL3.3 (Pin_3), R_F9.2
- new net CELL25: J_CELL3.2 (Pin_2), R_F8.2
- new net CELL26: J_CELL3.1 (Pin_1), R_F7.2
- new net CELL27: J_CELL4.6 (Pin_6), R_F6.2
- new net CELL28: J_CELL4.5 (Pin_5), R_F5.2
- new net CELL29: J_CELL4.4 (Pin_4), R_F4.2
- new net CELL3: J_CELL1.7 (Pin_7), R_F30.2
- new net CELL30: J_CELL4.3 (Pin_3), R_F3.2
- new net CELL31: J_CELL4.2 (Pin_2), R_F2.2
- new net CELL4: J_CELL1.6 (Pin_6), R_F29.2
- new net CELL5: J_CELL1.5 (Pin_5), R_F28.2
- new net CELL6: J_CELL1.4 (Pin_4), R_F27.2
- new net CELL7: J_CELL1.3 (Pin_3), R_F26.2
- new net CELL8: J_CELL1.2 (Pin_2), R_F25.2
- new net CELL9: J_CELL1.1 (Pin_1), R_F24.2
- new net CHG-: J_CHG1.2 (Pin_2), R_SH2.2
- new net SHUNT_MID: R_SH1.2, R_SH2.1
- no-connect marks 0 -> 40
Other:
- moved on the sheet: C_FLT1, C_SSR1, C_SSR2, Q1, Q2, R_B33, R_CHG1, R_G1, R_G2, R_SSR2, U_SSR1
